Commit message: Include holder and adjust camera transform

File: urdf/camera_gripper.xacro (robot description, xacro)
@@ -1,4 +1,32 @@
 <?xml version="1.0"?>
 <robot xmlns:xacro="http://www.ros.org/wiki/xacro" >
+    <joint name="zed2_holder_joint" type="fixed">
+        <parent link="panda_hand"/>
+        <child link="zed2_holder"/>
+        <origin xyz="0 0 0" rpy="${pi} 0 0"/>
+    </joint>
+    <link name="zed2_holder" >
+        <inertial>
+        <!-- Random values -->
+            <mass value="0.05"/>
+            <origin xyz="0 0 0"/>
+            <inertia
+                ixx="0.0003947" ixy="0.0" ixz="3.3365e-8"
+                iyy="2.417e-5" iyz="0.0"
+                izz="0.0003973"/>
+        </inertial>
+        <visual>
+            <geometry>
+                <mesh filename="package://franka_zed_gazebo/3d_prints/franka-ZED2-camera-holder.stl" scale="0.001 0.001 0.001"/>
+            </geometry>
+        </visual>
+        <!-- It was colliding with the robot at the mount point. Since it is not extremely relevant, collision was removed
+        <collision>
+            <geometry>
+                <mesh filename="package://franka_zed_gazebo/3d_prints/franka-ZED2-camera-holder.stl" scale="0.001 0.001 0.001"/>
+            </geometry>
+        </collision>
+        -->
+    </link>
     <joint name="camera_joint" type="fixed">
         <parent link="panda_hand"/>

File: urdf/camera_no_gripper.xacro (robot description, xacro)
@@ -1,8 +1,36 @@
 <?xml version="1.0"?>
 <robot xmlns:xacro="http://www.ros.org/wiki/xacro" >
+    <joint name="zed2_holder_joint" type="fixed">
+        <parent link="panda_hand"/>
+        <child link="zed2_holder"/>
+        <origin xyz="0 0 0" rpy="${pi} 0 0"/>
+    </joint>
+    <link name="zed2_holder" >
+        <inertial>
+        <!-- Random values -->
+            <mass value="0.05"/>
+            <origin xyz="0 0 0"/>
+            <inertia
+                ixx="0.0003947" ixy="0.0" ixz="3.3365e-8"
+                iyy="2.417e-5" iyz="0.0"
+                izz="0.0003973"/>
+        </inertial>
+        <visual>
+            <geometry>
+                <mesh filename="package://franka_zed_gazebo/3d_prints/franka-steep-ZED2-camera-holder.stl" scale="0.001 0.001 0.001"/>
+            </geometry>
+        </visual>
+        <!-- It was colliding with the robot at the mount point. Since it is not extremely relevant, collision was removed
+        <collision>
+            <geometry>
+                <mesh filename="package://franka_zed_gazebo/3d_prints/franka-steep-ZED2-camera-holder.stl" scale="0.001 0.001 0.001"/>
+            </geometry>
+        </collision>
+        -->
+    </link>
     <joint name="camera_joint" type="fixed">
         <parent link="panda_hand"/>
         <child link="camera_link"/>
-        <origin xyz="-0.097397 0 0.0274111" rpy="0 -1.35 0"/>
+        <origin xyz="-0.115 0 0.018" rpy="0 -1.35 0"/>
     </joint>
     <link name="camera_link">

File: urdf/panda_camera.urdf.xacro (robot description, xacro)
@@ -5,12 +5,9 @@
   Camera with MORE rotation relative to the end effector
   -->
-  <xacro:include filename="$(find franka_zed_gazebo)/urdf/camera_no_gripper.xacro" />
+  <xacro:include filename="$(find franka_zed_gazebo)/urdf/camera_gripper.xacro" />
   <!--
   Camera with LESS rotation relative to the end effector
   If you want the gripper to appear in the camera view, uncomment the following two lines and comment the one above
-  -->
-  <!--
   <xacro:include filename="$(find franka_zed_gazebo)/urdf/camera_gripper.xacro" />
-  <xacro:include filename="$(find franka_zed_gazebo)/urdf/zed2_holder_panda_gripper.xacro" />
   -->
   <xacro:arg name="arm_id" default="panda" />
